File: Power Supply Circuit Project/Fonte BDNM.kicad_pcb (KiCad board)
At the start: 2 copper layers, 96 x 113.5 mm, 15 parts, among them J1 + - DC Output, J2 Power In 18V AC 5A, SW1 Power Switch

Commit message: add files for milling
Parts:
- moved J1 2.67 mm to (41.8, 103.5)
Routing:
- net Net-(D1-+): track 238.5 -> 241.2 mm
Other:
- board text added: "+"
- board text added: "-"
- board text added: "bruno.pwn"
Changed lines of the file:
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@@
 			(disableapertmacros no)
 			(usegerberextensions no)
-			(usegerberattributes no)
-			(usegerberadvancedattributes no)
+			(usegerberattributes yes)
+			(usegerberadvancedattributes yes)
 			(creategerberjobfile yes)
 			(dashed_line_dash_ratio 12.000000)
@@
 		(pad "1" thru_hole circle
 			(at 0 0 90)
-			(size 1.6 1.6)
+			(size 2.5 2.5)
 			(drill 0.8)
 			(layers "*.Cu" "*.Mask")
@@
 		(pad "2" thru_hole circle
 			(at 5 0 90)
-			(size 1.6 1.6)
+			(size 2.5 2.5)
 			(drill 0.8)
 			(layers "*.Cu" "*.Mask")
@@
 	(footprint "TerminalBlock:TerminalBlock_MaiXu_MX126-5.0-02P_1x02_P5.00mm"
 		(layer "F.Cu")
-		(at 41.697315 100.802685)
+		(at 41.75 103.4675)
 		(descr "terminal block MaiXu MX126-5.0-02P, 2 pins, pitch 5mm, size 10.5x7.8mm, drill diameter 1.3mm, pad diameter 2.8mm, https://www.lcsc.com/datasheet/lcsc_datasheet_2309150913_MAX-MX126-5-0-03P-GN01-Cu-S-A_C5188435.pdf, script-generated using https://gitlab.com/kicad/libraries/kicad-footprint-generator/-/tree/master/scripts/TerminalBlock_MaiXu")
 		(tags "THT terminal block MaiXu MX126-5.0-02P pitch 5mm size 10.5x7.8mm drill 1.3mm pad 2.8mm")
@@
 		(pad "2" thru_hole circle
 			(at 7.5 0 90)
-			(size 2 2)
+			(size 2.5 2.5)
 			(drill 1)
 			(layers "*.Cu" "*.Mask")
@@
 		(pad "3" thru_hole circle
 			(at 15 0 90)
-			(size 2 2)
+			(size 2.5 2.5)
 			(drill 1)
 			(layers "*.Cu" "*.Mask")
@@
 		(pad "4" thru_hole circle
 			(at 25 0 90)
-			(size 2 2)
+			(size 2.5 2.5)
 			(drill 1)
 			(layers "*.Cu" "*.Mask")
@@
 		(pad "1" thru_hole circle
 			(at 0 0 270)
-			(size 1.6 1.6)
+			(size 2.5 2.5)
 			(drill 0.8)
 			(layers "*.Cu" "*.Mask")
@@
 		(pad "2" thru_hole circle
 			(at 5 0 270)
-			(size 1.6 1.6)
+			(size 2.5 2.5)
 			(drill 0.8)
 			(layers "*.Cu" "*.Mask")
@@
 		(pad "1" thru_hole oval
 			(at 0 0)
-			(size 3.25 6)
-			(drill 1.3)
+			(size 16.625 6)
+			(drill 1.3
+				(offset 6.6875 0)
+			)
 			(layers "*.Cu" "*.Mask")
 			(remove_unused_layers no)
@@
 		(pad "2" thru_hole oval
 			(at 37.5 0)
-			(size 3.25 6)
-			(drill 1.3)
+			(size 16.625 6)
+			(drill 1.3
+				(offset -6.6875 0)
+			)
 			(layers "*.Cu" "*.Mask")
 			(remove_unused_layers no)
@@
 		(pad "1" thru_hole circle
 			(at 0 0 90)
-			(size 1.6 1.6)
+			(size 2.5 2.5)
 			(drill 0.8)
 			(layers "*.Cu" "*.Mask")
@@
 		(pad "2" thru_hole circle
 			(at 5 0 90)
-			(size 1.6 1.6)
+			(size 2.5 2.5)
 			(drill 0.8)
 			(layers "*.Cu" "*.Mask")
@@
 		(pad "1" thru_hole circle
 			(at 0 0 270)
-			(size 1.6 1.6)
+			(size 2.5 2.5)
 			(drill 0.8)
 			(layers "*.Cu" "*.Mask")
@@
 		(pad "2" thru_hole circle
 			(at 5 0 270)
-			(size 1.6 1.6)
+			(size 2.5 2.5)
 			(drill 0.8)
 			(layers "*.Cu" "*.Mask")
@@
 		(pad "1" thru_hole circle
 			(at 0 0)
-			(size 1.6 1.6)
+			(size 2.5 2.5)
 			(drill 0.8)
 			(layers "*.Cu" "*.Mask")
@@
 		(pad "2" thru_hole circle
 			(at 7.62 0)
-			(size 1.6 1.6)
+			(size 2.5 2.5)
 			(drill 0.8)
 			(layers "*.Cu" "*.Mask")
@@
 		(pad "1" thru_hole circle
 			(at 0 0 90)
-			(size 1.8 1.8)
+			(size 2.5 2.5)
 			(drill 0.8)
 			(layers "*.Cu" "*.Mask")
@@
 		(pad "2" thru_hole circle
 			(at 7.5 2.9 90)
-			(size 1.8 1.8)
+			(size 2.5 2.5)
 			(drill 0.8)
 			(layers "*.Cu" "*.Mask")
@@
 		(layer "Edge.Cuts")
 	)
+	(gr_text "bruno.pwn"
+		(at 92.5 102 0)
+		(layer "B.Cu" knockout)
+		(effects
+			(font
+				(size 4.5 4.5)
+				(thickness 0.9)
+				(bold yes)
+			)
+			(justify left bottom mirror)
+		)
+	)
+	(gr_text "+"
+		(at 37.5 105 0)
+		(layer "B.Cu")
+		(effects
+			(font
+				(size 3 3)
+				(thickness 0.6)
+				(bold yes)
+			)
+			(justify left bottom mirror)
+		)
+	)
+	(gr_text "-"
+		(at 54 105 0)
+		(layer "B.Cu")
+		(effects
+			(font
+				(size 3 3)
+				(thickness 0.6)
+				(bold yes)
+			)
+			(justify left bottom mirror)
+		)
+	)
 	(segment
 		(start 78.697315 19.302685)
@@
 	)
 	(segment
-		(start 40.387315 91.302685)
-		(end 40.387315 99.492685)
+		(start 41.75 100.85537)
+		(end 41.75 103.4675)
 		(width 2)
 		(layer "B.Cu")
@@
 	)
 	(segment
-		(start 40.387315 99.492685)
-		(end 41.697315 100.802685)
+		(start 27.697315 71.802685)
+		(end 10.197315 71.802685)
 		(width 2)
 		(layer "B.Cu")
@@
 	)
 	(segment
-		(start 27.697315 71.802685)
-		(end 10.197315 71.802685)
+		(start 40.387315 91.302685)
+		(end 40.387315 99.492685)
 		(width 2)
 		(layer "B.Cu")
@@
 		(width 2)
 		(layer "B.Cu")
+		(net 2)
+	)
+	(segment
+		(start 40.387315 99.492685)
+		(end 41.75 100.85537)
+		(width 2)
+		(layer "B.Cu")
